Commit message: Remove AttrDict package dependency and fix mesh fille paths in .urdf files

File: data/urdf/tm5-900-hande.urdf (robot description, URDF)
Before this commit: robot tm5-900, 13 links, 12 joints
Links:
- link link_2: geometry collision mesh filename=../tm_description/meshes/tm5-900/collision/tm5-900_arm1_c.s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; visual mesh filename=../tm_description/meshes/tm5-900/visual/tm5-900_arm1.obj
- link link_4: geometry collision mesh filename=../tm_description/meshes/tm5-900/collision/tmr_100w_01_c.stl; visual mesh filename=../tm_description/meshes/tm5-900/visual/tmr_100w_01.obj
Joints:
- joint wrist_3_joint: origin xyz=0.000000 -0.113150 0.000000 rpy=1.570796 -0.000000 0.000000 -> xyz=0.000000 -0.113150 0.000000 rpy=1.570796 0.000000 0.000000
